File: Nonaddressable Controller.sch (EAGLE design)
At the start: 19 parts, among them IC1 PIC16F1826/27SO, K1 60V/32A/35mΩ, K2 60V/32A/35mΩ, K3 60V/32A/35mΩ, K4 60V/32A/35mΩ, K5 60V/32A/35mΩ, K6 60V/32A/35mΩ, X1 057-010-1

Commit message: Work on code for nonaddressable strip controller
Other:
- note added: "Blue"
- note added: "Green"
- note added: "Red"
Changed lines of the file:
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@@
 <sheet>
 <plain>
+<text x="-27.178" y="112.522" size="1.778" layer="97">Green</text>
+<text x="-34.798" y="108.712" size="1.778" layer="97">Red</text>
+<text x="-29.718" y="104.648" size="1.778" layer="97">Blue</text>
 </plain>
 <instances>
